Commit message: tb2

File: tb2/Assets/URDF/turtlebot2/robot_description.urdf (robot description, URDF)
Before this commit: robot turtlebot, 35 links, 34 joints
Links:
- removed link mount_xtion_pro_link
- link camera_link: mass 0.170 -> 0.564; geometry collision box size=0.0400 0.1650 0.0300; visual mesh filename=package://turtlebot_description/meshes/sensors/astra.dae scale=1 1 1
Joints:
- removed joint mount_xtion_pro_joint
- joint camera_depth_joint: origin xyz=0 0.027 0 rpy=0 0 0 -> xyz=0 0.025 0 rpy=0 0 0
- joint camera_depth_optical_joint: origin xyz=0 0 0 rpy=-1.57079632679 0 -1.57079632679 -> xyz=0 0 0 rpy=-1.5707963267948966 0 -1.5707963267948966
- joint camera_joint: origin xyz=0 -0.022 0 rpy=0 0 0 -> xyz=0 -0.0125 0 rpy=0 0 0
- joint camera_rgb_joint: origin xyz=-0.087 0.0205 0.287 rpy=0 0 0 -> xyz=-0.087 -0.0125 0.287 rpy=0 0 0
- joint camera_rgb_optical_joint: origin xyz=0 0 0 rpy=-1.57079632679 0 -1.57079632679 -> xyz=0 0 0 rpy=-1.5707963267948966 0 -1.5707963267948966
- joint caster_back_joint: origin xyz=-0.135 0.0 0.009 rpy=-1.57079632679 0 0 -> xyz=-0.135 0.0 0.009 rpy=-1.5707963267948966 0 0
- joint caster_front_joint: origin xyz=0.115 0.0 0.007 rpy=-1.57079632679 0 0 -> xyz=0.115 0.0 0.007 rpy=-1.5707963267948966 0 0
- joint cliff_sensor_front_joint: origin xyz=0.156 0.00 0.0214 rpy=0 1.57079632679 0 -> xyz=0.156 0.00 0.0214 rpy=0 1.5707963267948966 0
- joint cliff_sensor_left_joint: origin xyz=0.08734 0.13601 0.0214 rpy=0 1.57079632679 0 -> xyz=0.08734 0.13601 0.0214 rpy=0 1.5707963267948966 0
- joint cliff_sensor_right_joint: origin xyz=0.085 -0.13601 0.0214 rpy=0 1.57079632679 0 -> xyz=0.085 -0.13601 0.0214 rpy=0 1.5707963267948966 0
- joint wheel_left_joint: origin xyz=0.00 0.115 0.0250 rpy=-1.57079632679 0 0 -> xyz=0.00 0.115 0.0250 rpy=-1.5707963267948966 0 0
- joint wheel_right_joint: origin xyz=0.00 -0.115 0.0250 rpy=-1.57079632679 0 0 -> xyz=0.00 -0.115 0.0250 rpy=-1.5707963267948966 0 0
